File: Hardware/serial-mini/_autosave-serial-mini.sch (KiCad schematic (older format))
At the start: 52 parts, among them J1 PICKIT_V3_HEADER, J2 10118193-0001LF, J3 3-106505-2, Q1 IRLML2060, Q2 IRLML2060, Q3 IRLML2060, U1 SIT2001BI-S2-33S-100.000000D, U2 FT230XQ-R, U3 DSPIC33CK64MP105, U4 SN74AHC14RGYR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

Commit message: Update schematic symbols
Started adding schematic symbols to project specific library, mapping footprints to symbols
Parts:
- J1: value PICKIT_V3_HEADER -> PICKIT V3 Header
- J2: value 10118193-0001LF -> USB Micro B
- J3: value 3-106505-2 -> Serial Port
- U3: value DSPIC33CK64MP105 -> DSPIC33CK64MP102; symbol serial-mini:DSPIC33CK64MP105 -> serial-mini:DSPIC33CK64MP102
Changed lines of the file:
@@
 P 9950 3150
 F 0 "J1" V 9865 3728 45  0000 L CNN
-F 1 "PICKIT_V3_HEADER" V 9949 3728 45  0000 L CNN
+F 1 "PICKIT V3 Header" V 9949 3728 45  0000 L CNN
 F 2 "Connector_PinHeader_2.54mm:PinHeader_1x06_P2.54mm_Vertical" H 9950 3850 20  0001 C CNN
 F 3 "" H 9950 3150 50  0001 C CNN
@@
 $EndComp
 $Comp
-L serial-mini:DSPIC33CK64MP105 U3
+L serial-mini:DSPIC33CK64MP102 U3
 U 1 1 5D12D49B
 P 7200 4900
 F 0 "U3" H 7600 6415 50  0000 C CNN
-F 1 "DSPIC33CK64MP105" H 7600 6324 50  0000 C CNN
+F 1 "DSPIC33CK64MP102" H 7600 6324 50  0000 C CNN
 F 2 "serial-mini:‎DSPIC33CK32MP102" H 7200 4900 50  0001 C CNN
 F 3 "" H 7200 4900 50  0001 C CNN
@@
 P 10400 4700
 F 0 "J3" H 10928 4353 60  0000 L CNN
-F 1 "3-106505-2" H 10928 4247 60  0000 L CNN
+F 1 "Serial Port" H 10928 4247 60  0000 L CNN
 F 2 "serial-mini:3-106505-2" H 10800 4240 60  0001 C CNN
 F 3 "" H 10400 4700 60  0000 C CNN
@@
 P 11550 2600
 F 0 "Q1" H 11755 2600 50  0000 L CNN
-F 1 "IRLML2060" H 11754 2555 50  0001 L CNN
+F 1 "IRLML2060" H 11100 2750 50  0000 L CNN
 F 2 "serial-mini:IRLML2060TRPBF" H 11750 2700 50  0001 C CNN
 F 3 "~" H 11550 2600 50  0001 C CNN
@@
 P 11550 3300
 F 0 "Q2" H 11755 3300 50  0000 L CNN
-F 1 "IRLML2060" H 11754 3255 50  0001 L CNN
+F 1 "IRLML2060" H 11200 3450 50  0000 L CNN
 F 2 "serial-mini:IRLML2060TRPBF" H 11750 3400 50  0001 C CNN
 F 3 "~" H 11550 3300 50  0001 C CNN
@@
 P 11550 4000
 F 0 "Q3" H 11755 4000 50  0000 L CNN
-F 1 "IRLML2060" H 11754 3955 50  0001 L CNN
+F 1 "IRLML2060" H 11050 3900 50  0000 L CNN
 F 2 "serial-mini:IRLML2060TRPBF" H 11750 4100 50  0001 C CNN
 F 3 "~" H 11550 4000 50  0001 C CNN
@@
 P 13950 5850
 F 0 "J2" H 13842 5285 50  0000 C CNN
-F 1 "10118193-0001LF" H 13842 5376 50  0000 C CNN
+F 1 "USB Micro B" H 13842 5376 50  0000 C CNN
 F 2 "serial-mini:FCI_10118193-0001LF" H 13950 5850 50  0001 L BNN
 F 3 "" H 13950 5850 50  0001 L BNN
