File: Hardware/serial-mini/serial-mini.sch (KiCad schematic (older format))
At the start: 38 parts, among them J1 PICKIT_V3_HEADER, J2 10118193-0001LF, J5 10118193-0001LF, U1 SIT2001BI-S2-33S-100.000000D, U2 FT230XQ-R, U3 DSPIC33CK64MP105, U4 SN74AHC14RGYR, U5 MIC5504-3.3YMT-TZ

Commit message: Update schematic symbols
Started adding schematic symbols to project specific library, mapping footprints to symbols
Parts:
- removed C9: 0.1UF, Capacitor_SMD:C_0603_1608Metric, symbol serial-mini:10UF-0603-6.3V-20%
- removed J5: 10118193-0001LF, ps2mini:FCI_10118193-0001LF, symbol serial-mini:10118193-0001LF
- removed R7, R9: 10k, Resistor_SMD:R_0603_1608Metric, symbol ps2mini-rescue:RESISTOR0603-SparkFun-Resistors
- added D2, D3: LED, LED_SMD:LED_1210_3225Metric_Pad1.42x2.65mm_HandSolder, symbol serial-mini:SMD-LED-RGB(4P-0606)
- added D4: SMD-LED-RGB(4P-0606), LED_SMD:LED_1210_3225Metric_Pad1.42x2.65mm_HandSolder, symbol serial-mini:SMD-LED-RGB(4P-0606)
- added Q1, Q2, Q3: IRLML2060, serial-mini:IRLML2060TRPBF, symbol Device:Q_NMOS_GDS
- added R10, R12, R14: 130, Resistor_SMD:R_0603_1608Metric_Pad1.05x0.95mm_HandSolder, symbol serial-mini:RESISTOR0603
- added R11, R7, R9: 74, Resistor_SMD:R_0603_1608Metric_Pad1.05x0.95mm_HandSolder, symbol serial-mini:RESISTOR0603
- added R13, R15, R16, R17: 90, Resistor_SMD:R_0603_1608Metric_Pad1.05x0.95mm_HandSolder, symbol serial-mini:RESISTOR0603
- added R18, R19: 3352T-1-103LF, serial-mini:TRIM_3352T-1-103LF, symbol serial-mini:3352T-1-103LF
- C1, C10, C11, C12, C2, C3, C4, C5, C6, C7, C8: footprint Capacitor_SMD:C_0603_1608Metric -> Capacitor_SMD:C_0603_1608Metric_Pad1.05x0.95mm_HandSolder
- J1: footprint ps2mini:PinHeader_1x06_P2.54mm_Vertical -> Connector_PinHeader_2.54mm:PinHeader_1x06_P2.54mm_Vertical
- J2: footprint ps2mini:FCI_10118193-0001LF -> serial-mini:FCI_10118193-0001LF
- J3: renamed from J?; footprint CONN_3-106505-2_TYCO -> serial-mini:3-106505-2; symbol 2020-07-09_17-45-48:3-106505-2 -> serial-mini:3-106505-2
- R1, R2, R3, R4, R5, R6, R8: footprint Resistor_SMD:R_0603_1608Metric -> Resistor_SMD:R_0603_1608Metric_Pad1.05x0.95mm_HandSolder; symbol ps2mini-rescue:RESISTOR0603-SparkFun-Resistors -> serial-mini:RESISTOR0603
- S1, S2, S3: footprint ps2mini:Kailh_MX_Socket -> serial-mini:Kailh_MX_Socket
- U1: footprint ps2mini:SIT2001BI-S2-33S-100.000000D -> serial-mini:SIT2001BI-S2-33S-100.000000D
- U2: footprint ps2mini:QFN16 -> serial-mini:FT230XQ
- U3: value DSPIC33CK64MP105 -> DSPIC33CK64MP102; footprint ps2mini:QFN28 -> serial-mini:‎DSPIC33CK32MP102; symbol serial-mini:DSPIC33CK64MP105 -> serial-mini:DSPIC33CK64MP102
- U4: footprint ps2mini:SN74AHC14RGYR -> serial-mini:SN74AHC14RGYR
- U5: footprint ps2mini:VREG_MIC5504-3.3YMT-TZ -> serial-mini:MIC5504
Connections:
- net labels added: 57mA@1.7V, 69mA@1.7V, 69mA@3V
- net labels removed: SWITCH_OUT_4
- wire segments 119 -> 174
Other:
- moved on the sheet: C1, C10, C11, C12, C2, C3, C4, C5, C6, C7, C8, D1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

Commit message: Update symbols/footprints
Linked most symbols to their datasheets, updated more footprint/symbol footprints.
Also added status indicator LED
Parts:
- removed D1: RED LED, LED_SMD:LED_0603_1608Metric_Castellated, symbol Device:LED
- removed R17: 90, Resistor_SMD:R_0603_1608Metric_Pad1.05x0.95mm_HandSolder, symbol serial-mini:RESISTOR0603
- removed U5: MIC5504-3.3YMT-TZ, serial-mini:MIC5504, symbol serial-mini:MIC5504-3.3YMT-TZ
- added D?: LTST-C19FD1WT, 4-SMD, symbol serial-mini:LTST-C19FD1WT
- added R? (x2): 75, Resistor_SMD:R_0603_1608Metric_Pad1.05x0.95mm_HandSolder, symbol serial-mini:RESISTOR0603
- added R?: 50, Resistor_SMD:R_0603_1608Metric_Pad1.05x0.95mm_HandSolder, symbol serial-mini:RESISTOR0603
- added U?: MIC5504-3.3YM5-TR, SOT-23-5_MC_MCH, symbol serial-mini:MIC5504-3.3YM5-TR
- D2, D3, D4: Field4 HSMF-C118 -> (none)
- J1: value PICKIT_V3_HEADER -> PICKIT V3 Header; footprint Connector_PinHeader_2.54mm:PinHeader_1x06_P2.54mm_Vertical -> serial-mini:PICKITv3
- J2: value 10118193-0001LF -> USB Micro B; Field5 https://www.digikey.com/product-detail/en/amphenol-icc-fci/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 -> (none)
- J3: value 3-106505-2 -> Serial Port
- U2: Field7 https://www.digikey.com/product-detail/en/ftdi-future-techn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 -> (none)
Connections:
- net +3V3: now also U?.5 (VOUT)
- net +5V: now also D?.4, U?.1 (VIN), U?.3 (EN)
- net GND: now also U?.2 (GND)
- net at U3.RA1: now also R?.2
- net at U3.RA2: now also R?.2
- net at U3.RA3: now also R?.2
- new net: D?.1, R?.1
- new net: D?.2, R?.1
- new net: D?.3, R?.1
Other:
- moved on the sheet: C2
