File: Hardware/serial-mini.sch (KiCad schematic (older format))
At the start: 54 parts, among them J1 PICKIT V3 Header, J2 USB Micro B, J3 Serial Port, Q1 IRLML2060, Q2 IRLML2060, Q3 IRLML2060, U1 SIT2001BI-S2-33S-100.000000D, U2 FT230XQ-R, U3 DSPIC33CK64MP102, U4 SN74AHC14RGYR

Commit message: Add more labels
Swapped some LEDs
Parts:
- removed D?: LTST-C19FD1WT, 4-SMD, symbol serial-mini:LTST-C19FD1WT
- removed R? (x2): 75, Resistor_SMD:R_0603_1608Metric_Pad1.05x0.95mm_HandSolder, symbol serial-mini:RESISTOR0603
- removed R?: 50, Resistor_SMD:R_0603_1608Metric_Pad1.05x0.95mm_HandSolder, symbol serial-mini:RESISTOR0603
- added CR?: VAOL-S8WR4, LED_VCCLITE_0805_VCC, symbol serial-mini:VAOL-S8WR4
- added D?: LTST-C171KSKT, DIOC200X125X110, symbol serial-mini:LTST-C171KSKT
- added R?: 150, 0603, symbol serial-mini:RESISTOR0603-serial-mini
- added R?: 133, 0603, symbol serial-mini:RESISTOR0603-serial-mini
- R1, R10, R11, R12, R13, R14, R15, R16, R2, R3, R4, R5, R6, R7, R8, R9: symbol serial-mini:RESISTOR0603 -> serial-mini-rescue:RESISTOR0603-serial-mini
Connections:
- net labels added: 1.7V@57mA, 1.7V@69mA, 2V@15mA, 3V@20mA, 3V@69mA, Blue, Green, PWM-Brightness, PWM-Hue, RX, Red, TX
- net labels removed: 57mA@1.7V, 69mA@1.7V, 69mA@3V
- wire segments 179 -> 177
- no-connect marks 27 -> 24
Changed lines of the file:
@@
 $EndDescr
 $Comp
-L serial-mini:RESISTOR0603 R2
+L serial-mini-rescue:RESISTOR0603-serial-mini R2
 U 1 1 5D1378FB
 P 5050 7800
@@
 $EndComp
 $Comp
-L serial-mini:RESISTOR0603 R8
+L serial-mini-rescue:RESISTOR0603-serial-mini R8
 U 1 1 5D175B3E
 P 10250 3950
@@
 $EndComp
 $Comp
-L serial-mini:RESISTOR0603 R4
+L serial-mini-rescue:RESISTOR0603-serial-mini R4
 U 1 1 5D18CD99
 P 5700 7400
@@
 $EndComp
 $Comp
-L serial-mini:RESISTOR0603 R3
+L serial-mini-rescue:RESISTOR0603-serial-mini R3
 U 1 1 5D18DF88
 P 5400 7100
@@
 $EndComp
 $Comp
-L serial-mini:RESISTOR0603 R1
+L serial-mini-rescue:RESISTOR0603-serial-mini R1
 U 1 1 5D18FA64
 P 4700 8050
@@
 	8900 7500 8900 7600
 $Comp
-L serial-mini:RESISTOR0603 R6
+L serial-mini-rescue:RESISTOR0603-serial-mini R6
 U 1 1 5D1BFC28
 P 9500 7300
@@
 $EndComp
 $Comp
-L serial-mini:RESISTOR0603 R5
+L serial-mini-rescue:RESISTOR0603-serial-mini R5
 U 1 1 5D1BF50B
 P 9150 7600
@@
 NoConn ~ 11200 6100
 NoConn ~ 11200 6300
-NoConn ~ 11200 6500
 NoConn ~ 11200 6600
 NoConn ~ 11200 6700
@@
 Wire Wire Line
 	9000 6350 10800 6350
-Wire Wire Line
-	10800 6350 10800 5900
 Wire Wire Line
 	5750 4550 5900 4550
@@
 Wire Wire Line
 	9650 4800 10400 4800
-Text GLabel 11650 3800 0    50   Input ~ 0
-57mA@1.7V
 Wire Wire Line
 	12400 2150 12250 2150
@@
 	12900 2600 13050 2600
 $Comp
-L serial-mini:RESISTOR0603 R11
+L serial-mini-rescue:RESISTOR0603-serial-mini R11
 U 1 1 5F2CAB90
 P 12150 2950
@@
 Wire Wire Line
 	11850 2950 11850 2150
-Connection ~ 11850 2150
 Wire Wire Line
 	12800 4000 12900 4000
@@
 Connection ~ 12900 3300
 $Comp
-L serial-mini:RESISTOR0603 R9
+L serial-mini-rescue:RESISTOR0603-serial-mini R9
 U 1 1 5F2EC868
 P 12100 3650
@@
 	11750 3100 11650 3100
 $Comp
-L Device:Q_NMOS_GDS Q3
-U 1 1 5F302B1F
-P 11550 4000
-F 0 "Q3" H 11755 4000 50  0000 L CNN
-F 1 "IRLML2060" H 11050 3900 50  0000 L CNN
-F 2 "serial-mini:IRLML2060TRPBF" H 11750 4100 50  0001 C CNN
-F 3 "https://www.infineon.com/dgdl/irlml2060pbf.pdf?fileId=5546d462533600a401535664b7fb25ee" H 11550 4000 50  0001 C CNN
-	1    11550 4000
-	1    0    0    -1
-$EndComp
-$Comp
-L serial-mini:RESISTOR0603 R10
+L serial-mini-rescue:RESISTOR0603-serial-mini R10
 U 1 1 5F312013
 P 12150 2550
@@
 	11750 2550 11750 3050
 $Comp
-L serial-mini:RESISTOR0603 R12
+L serial-mini-rescue:RESISTOR0603-serial-mini R12
 U 1 1 5F31FB62
 P 12150 3300
@@
 $EndComp
 $Comp
-L serial-mini:RESISTOR0603 R14
+L serial-mini-rescue:RESISTOR0603-serial-mini R14
 U 1 1 5F3306F1
 P 12150 4000
@@
 	11750 3100 11750 4000
 $Comp
-L serial-mini:RESISTOR0603 R16
+L serial-mini-rescue:RESISTOR0603-serial-mini R16
 U 1 1 5F346C83
 P 12200 4300
@@
 	12400 4100 12400 4300
 $Comp
-L serial-mini:RESISTOR0603 R13
+L serial-mini-rescue:RESISTOR0603-serial-mini R13
 U 1 1 5F34E631
 P 12150 3450
@@
 	12400 3450 12350 3450
 $Comp
-L serial-mini:RESISTOR0603 R15
+L serial-mini-rescue:RESISTOR0603-serial-mini R15
 U 1 1 5F357E6E
 P 12200 2700
@@
 	1    0    0    -1
 $EndComp
-Text GLabel 11650 2150 0    50   Input ~ 0
-69mA@1.7V
 $Comp
 L power:+5V #PWR025
@@
 $EndComp
 $Comp
-L serial-mini:RESISTOR0603 R7
+L serial-mini-rescue:RESISTOR0603-serial-mini R7
 U 1 1 5F2A10BE
 P 12050 2150
@@
 	1    0    0    -1
 $EndComp
-Text GLabel 11750 3050 0    50   Input ~ 0
-69mA@3V
 Wire Wire Line
 	12600 6800 12600 7200
@@
 	7450 2850 7450 2700
 $Comp
-L serial-mini:LTST-C19FD1WT D?
-U 1 1 5F26AEEF
-P 5300 3950
-F 0 "D?" V 5717 4050 50  0000 C CNN
-F 1 "LTST-C19FD1WT" V 5626 4050 50  0000 C CNN
-F 2 "4-SMD" H 5300 3950 50  0001 L BNN
-F 3 "http://optoelectronics.liteon.com/upload/download/DS22-2001-076/LTST-C19FD1WT.pdf" H 5300 3950 50  0001 C CNN
-	1    5300 3950
-	0    -1   -1   0
-$EndComp
-$Comp
 L power:+5V #PWR?
 U 1 1 5F297A7B
-P 4400 3950
-F 0 "#PWR?" H 4400 3800 50  0001 C CNN
-F 1 "+5V" H 4415 4123 50  0000 C CNN
-F 2 "" H 4400 3950 50  0001 C CNN
-F 3 "" H 4400 3950 50  0001 C CNN
-	1    4400 3950
+P 4550 3750
+F 0 "#PWR?" H 4550 3600 50  0001 C CNN
+F 1 "+5V" H 4565 3923 50  0000 C CNN
+F 2 "" H 4550 3750 50  0001 C CNN
+F 3 "" H 4550 3750 50  0001 C CNN
+	1    4550 3750
 	0    -1   -1   0
 $EndComp
-Wire Wire Line
-	4400 3950 5000 3950
-$Comp
-L serial-mini:RESISTOR0603 R?
-U 1 1 5F2BDEC1
-P 5800 3750
-F 0 "R?" V 5705 3818 45  0000 L CNN
-F 1 "75" V 5789 3818 45  0000 L CNN
-F 2 "Resistor_SMD:R_0603_1608Metric_Pad1.05x0.95mm_HandSolder" H 5800 3900 20  0001 C CNN
-F 3 "" H 5800 3750 60  0001 C CNN
-F 4 " " V 5884 3818 60  0000 L CNN "Field4"
-	1    5800 3750
-	1    0    0    -1
-$EndComp
-$Comp
-L serial-mini:RESISTOR0603 R?
-U 1 1 5F2C26AE
-P 5800 3950
-F 0 "R?" V 5705 4018 45  0000 L CNN
-F 1 "50" V 5789 4018 45  0000 L CNN
-F 2 "Resistor_SMD:R_0603_1608Metric_Pad1.05x0.95mm_HandSolder" H 5800 4100 20  0001 C CNN
-F 3 "" H 5800 3950 60  0001 C CNN
-F 4 " " V 5884 4018 60  0000 L CNN "Field4"
-	1    5800 3950
-	1    0    0    -1
-$EndComp
-$Comp
-L serial-mini:RESISTOR0603 R?
-U 1 1 5F2C2BF1
-P 5800 4150
-F 0 "R?" V 5705 4218 45  0000 L CNN
-F 1 "75" V 5789 4218 45  0000 L CNN
-F 2 "Resistor_SMD:R_0603_1608Metric_Pad1.05x0.95mm_HandSolder" H 5800 4300 20  0001 C CNN
-F 3 "" H 5800 4150 60  0001 C CNN
-F 4 " " V 5884 4218 60  0000 L CNN "Field4"
-	1    5800 4150
-	1    0    0    -1
-$EndComp
-Wire Wire Line
-	5400 3750 5600 3750
-Wire Wire Line
-	6000 3750 6200 3750
-Wire Wire Line
-	6200 3950 6000 3950
-Wire Wire Line
-	5600 3950 5400 3950
-Wire Wire Line
-	5400 4150 5600 4150
-Wire Wire Line
-	6000 4150 6200 4150
 NoConn ~ 6200 5550
-NoConn ~ 10300 4550
-NoConn ~ 9850 4450
+Text Label 11650 2350 2    50   ~ 0
+1.7V@69mA
+Text Label 11750 3100 2    50   ~ 0
+3V@69mA
+Text Label 11650 3800 2    50   ~ 0
+1.7V@57mA
+$Comp
+L Device:Q_NMOS_GDS Q3
+U 1 1 5F302B1F
+P 11550 4000
+F 0 "Q3" H 11755 4000 50  0000 L CNN
+F 1 "IRLML2060" H 11050 3900 50  0000 L CNN
+F 2 "serial-mini:IRLML2060TRPBF" H 11750 4100 50  0001 C CNN
+F 3 "https://www.infineon.com/dgdl/irlml2060pbf.pdf?fileId=5546d462533600a401535664b7fb25ee" H 11550 4000 50  0001 C CNN
+	1    11550 4000
+	1    0    0    -1
+$EndComp
+Text Label 5350 5750 2    50   ~ 0
+PWM-Hue
+Text Label 9300 3500 2    50   ~ 0
+PWM-Brightness
+$Comp
+L serial-mini:VAOL-S8WR4 CR?
+U 1 1 5F2EDA7B
+P 5400 3750
+F 0 "CR?" H 5600 4138 60  0000 C CNN
+F 1 "VAOL-S8WR4" H 5600 4032 60  0000 C CNN
+F 2 "LED_VCCLITE_0805_VCC" H 5600 3390 60  0001 C CNN
+F 3 "http://vcclite.com/_pdf/VAOL-S8WR4-LED-0805-white.pdf" H 5600 4032 60  0001 C CNN
+	1    5400 3750
+	1    0    0    -1
+$EndComp
+Wire Wire Line
+	10800 5900 10800 6350
+$Comp
+L power:+5V #PWR?
+U 1 1 5F31F39B
+P 10050 6500
+F 0 "#PWR?" H 10050 6350 50  0001 C CNN
+F 1 "+5V" H 10065 6673 50  0000 C CNN
+F 2 "" H 10050 6500 50  0001 C CNN
+F 3 "" H 10050 6500 50  0001 C CNN
+	1    10050 6500
+	0    -1   1    0
+$EndComp
+$Comp
+L serial-mini:LTST-C171KSKT D?
+U 1 1 5F344729
+P 10700 6500
+F 0 "D?" H 10750 6283 50  0000 C CNN
+F 1 "LTST-C171KSKT" H 10750 6374 50  0000 C CNN
+F 2 "DIOC200X125X110" H 10700 6500 50  0001 L BNN
+F 3 "http://optoelectronics.liteon.com/upload/download/DS22-2000-110/LTST-C171KSKT.pdf" H 10700 6500 50  0001 L BNN
+	1    10700 6500
+	-1   0    0    1
+$EndComp
+$Comp
+L serial-mini:RESISTOR0603-serial-mini R?
+U 1 1 5F34B1D0
+P 10300 6500
+F 0 "R?" H 10300 6350 45  0000 C CNN
+F 1 "150" H 10300 6250 45  0000 C CNN
+F 2 "0603" H 10300 6650 20  0001 C CNN
+F 3 "" H 10300 6500 60  0001 C CNN
+F 4 " " H 10300 6621 60  0000 C CNN "Field4"
+	1    10300 6500
+	1    0    0    -1
+$EndComp
+Wire Wire Line
+	5800 3750 6200 3750
+$Comp
+L serial-mini:RESISTOR0603-serial-mini R?
+U 1 1 5F3D4344
+P 5050 3750
+F 0 "R?" H 5050 4050 45  0000 C CNN
+F 1 "133" H 5050 3966 45  0000 C CNN
+F 2 "0603" H 5050 3900 20  0001 C CNN
+F 3 "" H 5050 3750 60  0001 C CNN
+F 4 " " H 5050 3871 60  0000 C CNN "Field4"
+	1    5050 3750
+	1    0    0    -1
+$EndComp
+Wire Wire Line
+	5250 3750 5400 3750
+Wire Wire Line
+	4850 3750 4550 3750
+Wire Wire Line
+	10050 6500 10100 6500
+Wire Wire Line
+	10800 6500 11200 6500
+Text Label 10800 6500 0    50   ~ 0
+3V@20mA
+Text Label 5850 3750 0    50   ~ 0
+2V@15mA
+Text Label 9650 4550 0    50   ~ 0
+Green
+Text Label 9650 4350 0    50   ~ 0
+Red
+Text Label 9650 4150 0    50   ~ 0
+Blue
+Text Label 9200 4950 0    50   ~ 0
+RX
+Text Label 9200 5150 0    50   ~ 0
+TX
 $EndSCHEMATC

Commit message: Add test points
Swapped RGB LEDs, updated pin types to pass ERC, removed unused libraries/footprints
Parts:
- added TP-3.3V, TP-5V, TP-GND, TP1, TP10, TP2, TP3, TP4, TP6, TP8, TP9: TestPoint, TestPoint:TestPoint_Pad_1.0x1.0mm, symbol Connector:TestPoint
- added TP11, TP12, TP13, TP14, TP15, TP16, TP17, TP18: TestPoint, symbol Connector:TestPoint
- C1, C10, C11, C12, C2, C3, C4, C5, C6, C7, C8: symbol serial-mini:10UF-0603-6.3V-20% -> serial-mini:Capacitor
- D1: renamed from D?; footprint DIOC200X125X110 -> footprints:DIOC200X125X110
- D2, D3: footprint LED_SMD:LED_1210_3225Metric_Pad1.42x2.65mm_HandSolder -> footprints:CLVBA-FKA-CAEDH8BBB7A363
- D4: value SMD-LED-RGB(4P-0606) -> LED; footprint LED_SMD:LED_1210_3225Metric_Pad1.42x2.65mm_HandSolder -> footprints:CLVBA-FKA-CAEDH8BBB7A363
- D5: renamed from CR?; footprint LED_VCCLITE_0805_VCC -> footprints:VAOL-S8WR4
- J1: footprint serial-mini:PICKITv3 -> footprints:PICKITv3
- J2: footprint serial-mini:FCI_10118193-0001LF -> footprints:FCI_10118193-0001LF
- J3: footprint serial-mini:3-106505-2 -> footprints:3-106505-2
- Q1, Q2, Q3: footprint serial-mini:IRLML2060TRPBF -> footprints:IRLML2060TRPBF
- R1, R10, R11, R12, R13, R14, R15, R16, R2, R3, R4, R5, R6, R7, R8, R9: symbol serial-mini-rescue:RESISTOR0603-serial-mini -> serial-mini:Resistor
- R17, R20: renamed from R?; footprint 0603 -> Resistor_SMD:R_0603_1608Metric_Pad1.05x0.95mm_HandSolder
- R18, R19: footprint serial-mini:TRIM_3352T-1-103LF -> footprints:TRIM_3352T-1-103LF
- S1, S2, S3: footprint serial-mini:Kailh_MX_Socket -> footprints:Kailh_MX_Socket
- U1: footprint serial-mini:SIT2001BI-S2-33S-100.000000D -> footprints:SIT2001BI-S2-33S-100.000000D
- U2: footprint serial-mini:FT230XQ -> footprints:FT230XQ
- U3: footprint serial-mini:‎DSPIC33CK32MP102 -> footprints:‎DSPIC33CK32MP102
- U4: footprint serial-mini:SN74AHC14RGYR -> footprints:SN74AHC14RGYR
- U5: renamed from U?; footprint SOT-23-5_MC_MCH -> footprints:MIC5504
Connections:
- net +3V3: now also TP-3.3V.1
- net +5V: now also TP-5V.1
- net 1.7V@57mA: now also TP18.1
- net 1.7V@69mA: now also TP16.1
- net 2V@15mA: now also TP6.1
- net 3V@20mA: now also TP15.1
- net 3V@69mA: now also TP17.1
- net Blue: now also TP8.1
- net GND: now also TP-GND.1; no longer U4.15 (EPAD)
- net Green: now also TP10.1
- net PWM-Brightness: now also TP11.1
- net PWM-Hue: now also TP4.1
- net RX: now also TP13.1
- net Red: now also TP9.1
- net TX: now also TP14.1
- net at U1.5 (OUT), U3.RB0: now also TP1.1
- net at R3.2, R4.1, S2.2: now also TP2.1
- net at R5.2, R6.2, S3.1: now also TP12.1
- net at C4.1, R2.2, U4.5 (3A): now also TP3.1
- no-connect marks 24 -> 27

Commit message: Update PCB
Parts:
- TP-3.3V1: renamed from TP-3.3V; footprint TestPoint:TestPoint_Pad_1.0x1.0mm -> TestPoint:TestPoint_THTPad_1.0x1.0mm_Drill0.5mm
- TP-5V1: renamed from TP-5V; footprint TestPoint:TestPoint_Pad_1.0x1.0mm -> TestPoint:TestPoint_THTPad_1.0x1.0mm_Drill0.5mm
- TP-GND1: renamed from TP-GND; footprint TestPoint:TestPoint_Pad_1.0x1.0mm -> TestPoint:TestPoint_THTPad_1.0x1.0mm_Drill0.5mm
- TP1, TP10, TP2, TP3, TP4, TP6, TP8, TP9: footprint TestPoint:TestPoint_Pad_1.0x1.0mm -> TestPoint:TestPoint_THTPad_1.0x1.0mm_Drill0.5mm
- TP11, TP12, TP13, TP14, TP15, TP16, TP17, TP18: footprint (none) -> TestPoint:TestPoint_THTPad_1.0x1.0mm_Drill0.5mm
Connections:
- net USB_DM: now reaches J2.2 (D-), U2.7 (USBDM)
- net USB_DP: now reaches J2.3 (D+), U2.6 (USBDP)
Changed lines of the file:
@@
 TX
 $Comp
-L Connector:TestPoint TP-5V
+L Connector:TestPoint TP-5V1
 U 1 1 5F5E1403
 P 5700 2400
-F 0 "TP-5V" H 5758 2518 50  0000 L CNN
+F 0 "TP-5V1" H 5758 2518 50  0000 L CNN
 F 1 "TestPoint" H 5758 2427 50  0000 L CNN
-F 2 "TestPoint:TestPoint_Pad_1.0x1.0mm" H 5900 2400 50  0001 C CNN
+F 2 "TestPoint:TestPoint_THTPad_1.0x1.0mm_Drill0.5mm" H 5900 2400 50  0001 C CNN
 F 3 "~" H 5900 2400 50  0001 C CNN
 	1    5700 2400
@@
 	7450 2500 7650 2500
 $Comp
-L Connector:TestPoint TP-3.3V
+L Connector:TestPoint TP-3.3V1
 U 1 1 5F5FBCAA
 P 7450 2500
-F 0 "TP-3.3V" H 7508 2618 50  0000 L CNN
+F 0 "TP-3.3V1" H 7508 2618 50  0000 L CNN
 F 1 "TestPoint" H 7508 2527 50  0000 L CNN
-F 2 "TestPoint:TestPoint_Pad_1.0x1.0mm" H 7650 2500 50  0001 C CNN
+F 2 "TestPoint:TestPoint_THTPad_1.0x1.0mm_Drill0.5mm" H 7650 2500 50  0001 C CNN
 F 3 "~" H 7650 2500 50  0001 C CNN
 	1    7450 2500
@@
 F 0 "TP18" V 11845 3872 50  0000 C CNN
 F 1 "TestPoint" V 11754 3872 50  0000 C CNN
-F 2 "" H 11850 3800 50  0001 C CNN
+F 2 "TestPoint:TestPoint_THTPad_1.0x1.0mm_Drill0.5mm" H 11850 3800 50  0001 C CNN
 F 3 "~" H 11850 3800 50  0001 C CNN
 	1    11650 3800
@@
 F 0 "TP17" V 11845 3172 50  0000 C CNN
 F 1 "TestPoint" V 11754 3172 50  0000 C CNN
-F 2 "" H 11850 3100 50  0001 C CNN
+F 2 "TestPoint:TestPoint_THTPad_1.0x1.0mm_Drill0.5mm" H 11850 3100 50  0001 C CNN
 F 3 "~" H 11850 3100 50  0001 C CNN
 	1    11650 3100
@@
 F 0 "TP16" V 11845 2222 50  0000 C CNN
 F 1 "TestPoint" V 11754 2222 50  0000 C CNN
-F 2 "" H 11850 2150 50  0001 C CNN
+F 2 "TestPoint:TestPoint_THTPad_1.0x1.0mm_Drill0.5mm" H 11850 2150 50  0001 C CNN
 F 3 "~" H 11850 2150 50  0001 C CNN
 	1    11650 2150
@@
 F 0 "TP10" H 9192 4576 50  0000 R CNN
 F 1 "TestPoint" H 9192 4667 50  0000 R CNN
-F 2 "TestPoint:TestPoint_Pad_1.0x1.0mm" H 9450 4550 50  0001 C CNN
+F 2 "TestPoint:TestPoint_THTPad_1.0x1.0mm_Drill0.5mm" H 9450 4550 50  0001 C CNN
 F 3 "~" H 9450 4550 50  0001 C CNN
 	1    9250 4550
@@
 F 0 "TP9" H 9192 4376 50  0000 R CNN
 F 1 "TestPoint" H 9192 4467 50  0000 R CNN
-F 2 "TestPoint:TestPoint_Pad_1.0x1.0mm" H 9450 4350 50  0001 C CNN
+F 2 "TestPoint:TestPoint_THTPad_1.0x1.0mm_Drill0.5mm" H 9450 4350 50  0001 C CNN
 F 3 "~" H 9450 4350 50  0001 C CNN
 	1    9250 4350
@@
 F 0 "TP8" H 9192 4176 50  0000 R CNN
 F 1 "TestPoint" H 9192 4267 50  0000 R CNN
-F 2 "TestPoint:TestPoint_Pad_1.0x1.0mm" H 9450 4150 50  0001 C CNN
+F 2 "TestPoint:TestPoint_THTPad_1.0x1.0mm_Drill0.5mm" H 9450 4150 50  0001 C CNN
 F 3 "~" H 9450 4150 50  0001 C CNN
 	1    9250 4150
@@
 F 0 "TP2" H 5042 7426 50  0000 R CNN
 F 1 "TestPoint" H 5042 7517 50  0000 R CNN
-F 2 "TestPoint:TestPoint_Pad_1.0x1.0mm" H 5300 7400 50  0001 C CNN
+F 2 "TestPoint:TestPoint_THTPad_1.0x1.0mm_Drill0.5mm" H 5300 7400 50  0001 C CNN
 F 3 "~" H 5300 7400 50  0001 C CNN
 	1    5100 7400
@@
 F 0 "TP3" H 5508 7918 50  0000 L CNN
 F 1 "TestPoint" H 5508 7827 50  0000 L CNN
-F 2 "TestPoint:TestPoint_Pad_1.0x1.0mm" H 5650 7800 50  0001 C CNN
+F 2 "TestPoint:TestPoint_THTPad_1.0x1.0mm_Drill0.5mm" H 5650 7800 50  0001 C CNN
 F 3 "~" H 5650 7800 50  0001 C CNN
 	1    5450 7800
@@
 F 0 "TP12" H 9342 7626 50  0000 R CNN
 F 1 "TestPoint" H 9342 7717 50  0000 R CNN
-F 2 "" H 9600 7600 50  0001 C CNN
+F 2 "TestPoint:TestPoint_THTPad_1.0x1.0mm_Drill0.5mm" H 9600 7600 50  0001 C CNN
 F 3 "~" H 9600 7600 50  0001 C CNN
 	1    9400 7600
@@
 F 0 "TP15" H 10792 6526 50  0000 R CNN
 F 1 "TestPoint" H 10792 6617 50  0000 R CNN
-F 2 "" H 11050 6500 50  0001 C CNN
+F 2 "TestPoint:TestPoint_THTPad_1.0x1.0mm_Drill0.5mm" H 11050 6500 50  0001 C CNN
 F 3 "~" H 11050 6500 50  0001 C CNN
 	1    10850 6500
@@
 F 0 "TP6" H 5792 3776 50  0000 R CNN
 F 1 "TestPoint" H 5792 3867 50  0000 R CNN
-F 2 "TestPoint:TestPoint_Pad_1.0x1.0mm" H 6050 3750 50  0001 C CNN
+F 2 "TestPoint:TestPoint_THTPad_1.0x1.0mm_Drill0.5mm" H 6050 3750 50  0001 C CNN
 F 3 "~" H 6050 3750 50  0001 C CNN
 	1    5850 3750
@@
 F 0 "TP1" H 4558 5468 50  0000 L CNN
 F 1 "TestPoint" H 4558 5377 50  0000 L CNN
-F 2 "TestPoint:TestPoint_Pad_1.0x1.0mm" H 4700 5350 50  0001 C CNN
+F 2 "TestPoint:TestPoint_THTPad_1.0x1.0mm_Drill0.5mm" H 4700 5350 50  0001 C CNN
 F 3 "~" H 4700 5350 50  0001 C CNN
 	1    4500 5350
@@
 F 0 "TP4" H 5558 5868 50  0000 L CNN
 F 1 "TestPoint" H 5558 5777 50  0000 L CNN
-F 2 "TestPoint:TestPoint_Pad_1.0x1.0mm" H 5700 5750 50  0001 C CNN
+F 2 "TestPoint:TestPoint_THTPad_1.0x1.0mm_Drill0.5mm" H 5700 5750 50  0001 C CNN
 F 3 "~" H 5700 5750 50  0001 C CNN
 	1    5500 5750
@@
 F 0 "TP11" V 9254 3938 50  0000 L CNN
 F 1 "TestPoint" V 9345 3938 50  0000 L CNN
-F 2 "" H 9500 3750 50  0001 C CNN
+F 2 "TestPoint:TestPoint_THTPad_1.0x1.0mm_Drill0.5mm" H 9500 3750 50  0001 C CNN
 F 3 "~" H 9500 3750 50  0001 C CNN
 	1    9300 3750
@@
 F 0 "TP13" H 9508 5068 50  0000 L CNN
 F 1 "TestPoint" H 9508 4977 50  0000 L CNN
-F 2 "" H 9650 4950 50  0001 C CNN
+F 2 "TestPoint:TestPoint_THTPad_1.0x1.0mm_Drill0.5mm" H 9650 4950 50  0001 C CNN
 F 3 "~" H 9650 4950 50  0001 C CNN
 	1    9450 4950
@@
 F 0 "TP14" H 9508 5268 50  0000 L CNN
 F 1 "TestPoint" H 9508 5177 50  0000 L CNN
-F 2 "" H 9650 5150 50  0001 C CNN
+F 2 "TestPoint:TestPoint_THTPad_1.0x1.0mm_Drill0.5mm" H 9650 5150 50  0001 C CNN
 F 3 "~" H 9650 5150 50  0001 C CNN
 	1    9450 5150
@@
 $EndComp
 $Comp
-L Connector:TestPoint TP-GND
+L Connector:TestPoint TP-GND1
 U 1 1 5F8BEC1A
 P 5300 2900
-F 0 "TP-GND" H 5358 3018 50  0000 L CNN
+F 0 "TP-GND1" H 5358 3018 50  0000 L CNN
 F 1 "TestPoint" H 5358 2927 50  0000 L CNN
-F 2 "TestPoint:TestPoint_Pad_1.0x1.0mm" H 5500 2900 50  0001 C CNN
+F 2 "TestPoint:TestPoint_THTPad_1.0x1.0mm_Drill0.5mm" H 5500 2900 50  0001 C CNN
 F 3 "~" H 5500 2900 50  0001 C CNN
 	1    5300 2900
@@
 Wire Wire Line
 	5300 2900 5300 2800
+Text Label 12700 6050 0    50   ~ 0
+USB_DM
+Text Label 12700 6100 0    50   ~ 0
+USB_DP
 $EndSCHEMATC
