File: Hardware/regulator.sch (KiCad schematic (older format))
At the start: 6 parts, among them U4 MIC5504-3.3YM5-TR

Commit message: Complete new schematic
Added MAX232 and fixed test points on switches
Parts:
- TP-3.3V1, TP-5V1, TP-GND1: footprint TestPoint:TestPoint_Pad_1.0x1.0mm -> TestPoint:TestPoint_THTPad_1.0x1.0mm_Drill0.5mm
Changed lines of the file:
@@
 F 0 "TP-5V1" H 5008 3868 50  0000 L CNN
 F 1 "TestPoint" H 5008 3777 50  0000 L CNN
-F 2 "TestPoint:TestPoint_Pad_1.0x1.0mm" H 5150 3750 50  0001 C CNN
+F 2 "TestPoint:TestPoint_THTPad_1.0x1.0mm_Drill0.5mm" H 5150 3750 50  0001 C CNN
 F 3 "~" H 5150 3750 50  0001 C CNN
 	1    4950 3750
@@
 F 0 "TP-3.3V1" H 6758 3968 50  0000 L CNN
 F 1 "TestPoint" H 6758 3877 50  0000 L CNN
-F 2 "TestPoint:TestPoint_Pad_1.0x1.0mm" H 6900 3850 50  0001 C CNN
+F 2 "TestPoint:TestPoint_THTPad_1.0x1.0mm_Drill0.5mm" H 6900 3850 50  0001 C CNN
 F 3 "~" H 6900 3850 50  0001 C CNN
 	1    6700 3850
@@
 F 0 "TP-GND1" H 4608 4368 50  0000 L CNN
 F 1 "TestPoint" H 4608 4277 50  0000 L CNN
-F 2 "TestPoint:TestPoint_Pad_1.0x1.0mm" H 4750 4250 50  0001 C CNN
+F 2 "TestPoint:TestPoint_THTPad_1.0x1.0mm_Drill0.5mm" H 4750 4250 50  0001 C CNN
 F 3 "~" H 4750 4250 50  0001 C CNN
 	1    4550 4250
