File: Hardware/power-regulator.sch (KiCad schematic (older format))
At the start: 6 parts, among them U4 MIC5504-3.3YM5-TR

Commit message: Fix faulty debounce circuit
Used wrong value resistor/misplaced on each switch.
Also adjusted value of RC circuits for a time constant of 1 microsecond (was 1 millisecond before)
Parts:
- TP-3.3V1, TP-5V1, TP-GND1: footprint TestPoint:TestPoint_THTPad_1.0x1.0mm_Drill0.5mm -> TestPoint:TestPoint_Pad_1.0x1.0mm
Changed lines of the file:
@@
 F 0 "TP-5V1" H 5208 3868 50  0000 L CNN
 F 1 "TestPoint" H 5208 3777 50  0000 L CNN
-F 2 "TestPoint:TestPoint_THTPad_1.0x1.0mm_Drill0.5mm" H 5350 3750 50  0001 C CNN
+F 2 "TestPoint:TestPoint_Pad_1.0x1.0mm" H 5350 3750 50  0001 C CNN
 F 3 "~" H 5350 3750 50  0001 C CNN
 	1    5150 3750
@@
 F 0 "TP-3.3V1" H 6958 3968 50  0000 L CNN
 F 1 "TestPoint" H 6958 3877 50  0000 L CNN
-F 2 "TestPoint:TestPoint_THTPad_1.0x1.0mm_Drill0.5mm" H 7100 3850 50  0001 C CNN
+F 2 "TestPoint:TestPoint_Pad_1.0x1.0mm" H 7100 3850 50  0001 C CNN
 F 3 "~" H 7100 3850 50  0001 C CNN
 	1    6900 3850
@@
 F 0 "TP-GND1" H 4808 4368 50  0000 L CNN
 F 1 "TestPoint" H 4808 4277 50  0000 L CNN
-F 2 "TestPoint:TestPoint_THTPad_1.0x1.0mm_Drill0.5mm" H 4950 4250 50  0001 C CNN
+F 2 "TestPoint:TestPoint_Pad_1.0x1.0mm" H 4950 4250 50  0001 C CNN
 F 3 "~" H 4950 4250 50  0001 C CNN
 	1    4750 4250
