File: Hardware/rs232-converter.sch (KiCad schematic (older format))
At the start: 8 parts, among them J3 Serial Port, U1 MAX232

Commit message: Complete new schematic
Added MAX232 and fixed test points on switches
Parts:
- U1: footprint (none) -> footprints:MAX232ECPWR
Connections:
- no-connect marks 12 -> 11
Other:
- moved on the sheet: TP12
Changed lines of the file:
@@
 L Connector:TestPoint TP?
 U 1 1 5F838235
-P 7500 3900
+P 7550 4300
 AR Path="/5F838235" Ref="TP?"  Part="1"
 AR Path="/5F821E36/5F838235" Ref="TP12"  Part="1"
-F 0 "TP12" H 7600 4100 50  0000 L CNN
-F 1 "TestPoint" H 7600 4000 50  0000 L CNN
-F 2 "TestPoint:TestPoint_THTPad_1.0x1.0mm_Drill0.5mm" H 7700 3900 50  0001 C CNN
-F 3 "~" H 7700 3900 50  0001 C CNN
-	1    7500 3900
+F 0 "TP12" H 7650 4500 50  0000 L CNN
+F 1 "TestPoint" H 7650 4400 50  0000 L CNN
+F 2 "TestPoint:TestPoint_THTPad_1.0x1.0mm_Drill0.5mm" H 7750 4300 50  0001 C CNN
+F 3 "~" H 7750 4300 50  0001 C CNN
+	1    7550 4300
 	1    0    0    -1
 $EndComp
@@
 F 0 "U1" H 6600 4981 50  0000 C CNN
 F 1 "MAX232" H 6600 4890 50  0000 C CNN
-F 2 "" H 6650 2550 50  0001 L CNN
+F 2 "footprints:MAX232ECPWR" H 6650 2550 50  0001 L CNN
 F 3 "http://www.ti.com/lit/ds/symlink/max232.pdf" H 6600 3700 50  0001 C CNN
 	1    6600 3600
@@
 Wire Wire Line
 	7550 4400 7950 4400
-Connection ~ 7500 3900
 Wire Wire Line
-	7500 4300 7950 4300
+	7500 4300 7550 4300
 Text HLabel 5800 3900 0    50   Input ~ 0
 TX-Serial-Port
@@
 NoConn ~ 7400 3700
 NoConn ~ 7400 4100
-NoConn ~ 7800 3650
 $Comp
 L power:+5V #PWR?
@@
 	1    0    0    -1
 $EndComp
+Connection ~ 7550 4300
+Wire Wire Line
+	7550 4300 7950 4300
 $EndSCHEMATC

Commit message: Add more net labels
Begin redesigning PCB again
Connections:
- net RS232-RX: now reaches J3.2, TP12.1, U1.7 (T2OUT)
- net RS232-TX: now reaches J3.3, TP13.1, U1.8 (R2IN)
- net RX-Serial-Port renamed Serial-Port-RX
- net TX-Serial-Port renamed Serial-Port-TX
Changed lines of the file:
@@
 $Descr A4 11693 8268
 encoding utf-8
-Sheet 7 7
+Sheet 6 7
 Title ""
 Date ""
@@
 	7500 4300 7550 4300
 Text HLabel 5800 3900 0    50   Input ~ 0
-TX-Serial-Port
+Serial-Port-TX
 Text HLabel 5800 4300 0    50   Input ~ 0
-RX-Serial-Port
+Serial-Port-RX
 $Comp
 L serial-mini:Capacitor C?
@@
 Wire Wire Line
 	7550 4300 7950 4300
+Text Label 7550 4400 0    50   ~ 0
+RS232-TX
+Text Label 7550 4300 0    50   ~ 0
+RS232-RX
 $EndSCHEMATC

Commit message: Fix faulty debounce circuit
Used wrong value resistor/misplaced on each switch.
Also adjusted value of RC circuits for a time constant of 1 microsecond (was 1 millisecond before)
Parts:
- TP12, TP13: footprint TestPoint:TestPoint_THTPad_1.0x1.0mm_Drill0.5mm -> TestPoint:TestPoint_Pad_1.0x1.0mm
Changed lines of the file:
@@
 F 0 "TP13" H 7600 4700 50  0000 L CNN
 F 1 "TestPoint" H 7550 4600 50  0000 L CNN
-F 2 "TestPoint:TestPoint_THTPad_1.0x1.0mm_Drill0.5mm" H 7750 4400 50  0001 C CNN
+F 2 "TestPoint:TestPoint_Pad_1.0x1.0mm" H 7750 4400 50  0001 C CNN
 F 3 "~" H 7750 4400 50  0001 C CNN
 	1    7550 4400
@@
 F 0 "TP12" H 7650 4500 50  0000 L CNN
 F 1 "TestPoint" H 7650 4400 50  0000 L CNN
-F 2 "TestPoint:TestPoint_THTPad_1.0x1.0mm_Drill0.5mm" H 7750 4300 50  0001 C CNN
+F 2 "TestPoint:TestPoint_Pad_1.0x1.0mm" H 7750 4300 50  0001 C CNN
 F 3 "~" H 7750 4300 50  0001 C CNN
 	1    7550 4300

Commit message: Add BOM
Parts:
- J3: value Serial Port -> 3-106505-2
- U1: value MAX232 -> MAX232ECPWR
Changed lines of the file:
@@
 AR Path="/5F821E36/5F838222" Ref="J3"  Part="1"
 F 0 "J3" H 8478 3853 60  0000 L CNN
-F 1 "Serial Port" H 8478 3747 60  0000 L CNN
+F 1 "3-106505-2" H 8478 3747 60  0000 L CNN
 F 2 "footprints:3-106505-2" H 8350 3740 60  0001 C CNN
 F 3 "https://www.te.com/commerce/DocumentDelivery/DDEController?Action=srchrtrv&DocNm=82068_AMPLIMITE_Right-Angle_Posted_Conn&DocType=CS&DocLang=English" H 7950 4200 60  0001 C CNN
@@
 AR Path="/5F821E36/5F838243" Ref="U1"  Part="1"
 F 0 "U1" H 6600 4981 50  0000 C CNN
-F 1 "MAX232" H 6600 4890 50  0000 C CNN
+F 1 "MAX232ECPWR" H 6600 4890 50  0000 C CNN
 F 2 "footprints:MAX232ECPWR" H 6650 2550 50  0001 L CNN
 F 3 "http://www.ti.com/lit/ds/symlink/max232.pdf" H 6600 3700 50  0001 C CNN
