File: Hardware/usb-uart.sch (KiCad schematic (older format))
At the start: 16 parts, among them J2 USB Micro B, U6 FT230XQ-R

Commit message: Complete new schematic
Added MAX232 and fixed test points on switches
Parts:
- removed C9: 10uF, Capacitor_SMD:C_0603_1608Metric_Pad1.05x0.95mm_HandSolder, symbol serial-mini:Capacitor
- FB1: footprint (none) -> Resistor_SMD:R_0805_2012Metric_Pad1.15x1.40mm_HandSolder
Changed lines of the file:
@@
 F 0 "FB1" H 8600 4796 50  0000 L CNN
 F 1 "Ferrite_Bead_Small" H 8600 4705 50  0000 L CNN
-F 2 "" V 8430 4750 50  0001 C CNN
+F 2 "Resistor_SMD:R_0805_2012Metric_Pad1.15x1.40mm_HandSolder" V 8430 4750 50  0001 C CNN
 F 3 "~" H 8500 4750 50  0001 C CNN
 	1    8500 4750
@@
 NoConn ~ 3250 3700
 NoConn ~ 3250 3500
-Wire Wire Line
-	4700 2400 4700 2600
 $Comp
 L power:GND #PWR?
-U 1 1 5F793703
-P 4700 2400
-AR Path="/5F793703" Ref="#PWR?"  Part="1"
-AR Path="/5F78F2B4/5F793703" Ref="#PWR034"  Part="1"
-F 0 "#PWR034" H 4700 2150 50  0001 C CNN
-F 1 "GND" H 4705 2227 50  0000 C CNN
-F 2 "" H 4700 2400 50  0001 C CNN
-F 3 "" H 4700 2400 50  0001 C CNN
-	1    4700 2400
-	1    0    0    1
-$EndComp
-Connection ~ 4700 3100
-Wire Wire Line
-	4700 2900 4700 3100
-$Comp
-L serial-mini:Capacitor C?
-U 1 1 5F79370C
-P 4700 2700
-AR Path="/5F79370C" Ref="C?"  Part="1"
-AR Path="/5F78F2B4/5F79370C" Ref="C9"  Part="1"
-F 0 "C9" V 4550 2700 45  0000 C CNN
-F 1 "10uF" V 4550 2850 45  0000 C CNN
-F 2 "Capacitor_SMD:C_0603_1608Metric_Pad1.05x0.95mm_HandSolder" H 4700 2950 20  0001 C CNN
-F 3 "" H 4700 2700 50  0001 C CNN
-F 4 "" H 4808 2666 60  0000 L CNN "Field4"
-	1    4700 2700
-	1    0    0    1
-$EndComp
-$Comp
-L power:GND #PWR?

Commit message: Add more net labels
Begin redesigning PCB again
Connections:
- net D+: now reaches D6.1 (I/O1), J2.3 (D+)
- net Shield: now reaches C14.2, D6.2 (GND), J2.S1 (SHIELD), J2.S2 (SHIELD), J2.S3 (SHIELD), J2.S4 (SHIELD), J2.S5 (SHIELD), J2.S6 (SHIELD), R23.1
- net D-: now reaches D6.3 (I/O2), J2.2 (D-)
- net RX-USB renamed USB-RX
- net TX-USB renamed USB-TX
Changed lines of the file:
@@
 $Descr A4 11693 8268
 encoding utf-8
-Sheet 6 7
+Sheet 5 7
 Title ""
 Date ""
@@
 $EndComp
 Text HLabel 2700 3100 0    50   Input ~ 0
-RX-USB
+USB-RX
 Text HLabel 2700 3300 0    50   Input ~ 0
-TX-USB
+USB-TX
 Wire Wire Line
 	3250 3100 2700 3100
@@
 Text Label 8500 4100 2    50   ~ 0
 VUSB
+Text Label 8200 3750 0    50   ~ 0
+D+
+Text Label 8200 3850 0    50   ~ 0
+D-
+Text Label 7650 2650 0    50   ~ 0
+Shield
 $EndSCHEMATC

Commit message: Complete initial routing
Parts:
- removed J2: USB Micro B, footprints:AMPHENOL_10103593-0001LF, symbol serial-mini:10118193-0001LF
- added J2: 10103593-0001LF, footprints:AMPHENOL_10103593-0001LF, symbol serial-mini:10103593-0001LF
Connections:
- net D+: now also J2.3 (D+)
- net D-: now also J2.2 (D-)
- net GND: now also J2.5 (GND)
- net Shield: now also J2.S1 (SHIELD), J2.S2 (SHIELD), J2.S3 (SHIELD), J2.S4 (SHIELD), J2.S5 (SHIELD), J2.S6 (SHIELD)
- net VUSB: now also J2.1 (VCC)
Changed lines of the file:
@@
 Text Label 2850 3900 0    50   ~ 0
 3V@20mA
-$Comp
-L serial-mini:10118193-0001LF J?
-U 1 1 5F7936DD
-P 9000 3650
-AR Path="/5F7936DD" Ref="J?"  Part="1"
-AR Path="/5F78F2B4/5F7936DD" Ref="J2"  Part="1"
-F 0 "J2" H 8892 3085 50  0000 C CNN
-F 1 "USB Micro B" H 8892 3176 50  0000 C CNN
-F 2 "footprints:AMPHENOL_10103593-0001LF" H 9000 3650 50  0001 L BNN
-F 3 "https://www.digikey.com/product-detail/en/amphenol-icc-fci/10118193-0001LF/609-4616-1-ND/2785380?utm_source=snapeda&utm_medium=aggregator&utm_campaign=symbol" H 9000 3650 50  0001 L BNN
-F 4 "None" H 9000 3650 50  0001 L BNN "Field4"
-F 5 "" H 9000 3650 50  0001 L BNN "Field5"
-F 6 "10118193-0001LF" H 9000 3650 50  0001 L BNN "Field6"
-F 7 "Amphenol ICC" H 9000 3650 50  0001 L BNN "Field7"
-F 8 "609-4616-1-ND" H 9000 3650 50  0001 L BNN "Field8"
-	1    9000 3650
-	1    0    0    1
-$EndComp
 Wire Wire Line
 	4650 4200 4650 3900
@@
 Text Label 7650 2650 0    50   ~ 0
 Shield
+$Comp
+L serial-mini:10103593-0001LF J2
+U 1 1 5F23D588
+P 9000 3750
+F 0 "J2" H 9230 3796 50  0000 L CNN
+F 1 "10103593-0001LF" H 9230 3705 50  0000 L CNN
+F 2 "footprints:AMPHENOL_10103593-0001LF" H 9000 3750 50  0001 L BNN
+F 3 "2.99mm" H 9000 3750 50  0001 L BNN
+F 4 "Amphenol FCI" H 9000 3750 50  0001 L BNN "Field4"
+F 5 "A" H 9000 3750 50  0001 L BNN "Field5"
+F 6 "Manufacturer Recommendations" H 9000 3750 50  0001 L BNN "Field6"
+	1    9000 3750
+	1    0    0    -1
+$EndComp
 $EndSCHEMATC

Commit message: Fix faulty debounce circuit
Used wrong value resistor/misplaced on each switch.
Also adjusted value of RC circuits for a time constant of 1 microsecond (was 1 millisecond before)
Parts:
- TP11: footprint TestPoint:TestPoint_THTPad_1.0x1.0mm_Drill0.5mm -> TestPoint:TestPoint_Pad_1.0x1.0mm
Changed lines of the file:
@@
 Wire Wire Line
 	8500 3950 8500 4400
-Wire Wire Line
-	8500 4650 8500 4400
 Connection ~ 8500 4400
 $Comp
@@
 	1    8400 4400
 	0    -1   1    0
-$EndComp
-$Comp
-L Device:Ferrite_Bead_Small FB?
-U 1 1 5F793686
-P 8500 4750
-AR Path="/5F793686" Ref="FB?"  Part="1"
-AR Path="/5F78F2B4/5F793686" Ref="FB1"  Part="1"
-F 0 "FB1" H 8600 4796 50  0000 L CNN
-F 1 "Ferrite_Bead_Small" H 8600 4705 50  0000 L CNN
-F 2 "Resistor_SMD:R_0805_2012Metric_Pad1.15x1.40mm_HandSolder" V 8430 4750 50  0001 C CNN
-F 3 "~" H 8500 4750 50  0001 C CNN
-	1    8500 4750
-	1    0    0    -1
 $EndComp
 $Comp
@@
 F 1 "FT230XQ-R" H 3950 4679 50  0000 C CNN
 F 2 "footprints:FT230XQ" H 3950 3800 50  0001 L BNN
-F 3 "https://www.digikey.com/product-detail/en/ftdi-future-technology-devices-international-ltd/FT230XQ-R/768-1130-1-ND/3029158?utm_source=snapeda&utm_medium=aggregator&utm_campaign=symbol" H 3950 3800 50  0001 L BNN
+F 3 "https://www.ftdichip.com/Support/Documents/DataSheets/ICs/DS_FT230X.pdf" H 3950 3800 50  0001 L BNN
 F 4 "768-1130-1-ND" H 3950 3800 50  0001 L BNN "Field4"
 F 5 "QFN-16 FTDI" H 3950 3800 50  0001 L BNN "Field5"
@@
 F 0 "TP11" H 2842 3926 50  0000 R CNN
 F 1 "TestPoint" H 2842 4017 50  0000 R CNN
-F 2 "TestPoint:TestPoint_THTPad_1.0x1.0mm_Drill0.5mm" H 3100 3900 50  0001 C CNN
+F 2 "TestPoint:TestPoint_Pad_1.0x1.0mm" H 3100 3900 50  0001 C CNN
 F 3 "~" H 3100 3900 50  0001 C CNN
 	1    2900 3900
@@
 	1    0    0    -1
 $EndComp
+Wire Wire Line
+	8500 4650 8500 4400
+$Comp
+L Device:Ferrite_Bead_Small FB?
+U 1 1 5F793686
+P 8500 4750
+AR Path="/5F793686" Ref="FB?"  Part="1"
+AR Path="/5F78F2B4/5F793686" Ref="FB1"  Part="1"
+F 0 "FB1" H 8600 4796 50  0000 L CNN
+F 1 "Ferrite_Bead_Small" H 8600 4705 50  0000 L CNN
+F 2 "Resistor_SMD:R_0805_2012Metric_Pad1.15x1.40mm_HandSolder" V 8430 4750 50  0001 C CNN
+F 3 "~" H 8500 4750 50  0001 C CNN
+	1    8500 4750
+	1    0    0    -1
+$EndComp

Commit message: Add BOM
Parts:
- FB1: value Ferrite_Bead_Small -> MI0805K601R
Changed lines of the file:
@@
 AR Path="/5F78F2B4/5F793686" Ref="FB1"  Part="1"
 F 0 "FB1" H 8600 4796 50  0000 L CNN
-F 1 "Ferrite_Bead_Small" H 8600 4705 50  0000 L CNN
+F 1 "MI0805K601R" H 8600 4705 50  0000 L CNN
 F 2 "Resistor_SMD:R_0805_2012Metric_Pad1.15x1.40mm_HandSolder" V 8430 4750 50  0001 C CNN
 F 3 "~" H 8500 4750 50  0001 C CNN

Commit message: Fix PRTR5V0U2F footprint
Footprint was flipped wrong way on PCB, also removed BOM folder since it messed up Linguist
Connections:
- net D+: now also D6.3 (I/O2); no longer D6.1 (I/O1)
- net D-: now also D6.1 (I/O1); no longer D6.3 (I/O2)
- net at C12.2, D6.4 (I/O2): now also R22.2; no longer R21.2
- net at C13.1, D6.6 (I/O1): now also R21.2; no longer R22.2
Changed lines of the file:
@@
 	1    0    0    1
 $EndComp
-Wire Wire Line
-	5550 2900 5850 2900
 $Comp
 L serial-mini:Capacitor C?
@@
 Wire Wire Line
 	5550 4300 5300 4300
-Wire Wire Line
-	5550 3900 5850 3900
-Wire Wire Line
-	5550 4000 5550 3900
 $Comp
 L serial-mini:Capacitor C?
@@
 	-1   0    0    -1
 $EndComp
-Connection ~ 5550 3900
-Wire Wire Line
-	5250 3900 5550 3900
-Wire Wire Line
-	5250 3500 5250 3900
-Connection ~ 5550 2900
-Wire Wire Line
-	5250 2900 5550 2900
-Wire Wire Line
-	5250 3300 5250 2900
 Wire Wire Line
 	4650 3500 4850 3500
@@
 Wire Wire Line
 	8200 2650 7350 2650
-Wire Wire Line
-	7650 2900 7050 2900
-Wire Wire Line
-	7650 3850 7650 2900
-Wire Wire Line
-	7050 3900 8100 3900
 $Comp
 L serial-mini:PRTR5V0U2F,115 D?
@@
 $EndComp
 Wire Wire Line
-	8600 3850 7650 3850
-Wire Wire Line
-	8100 3750 8100 3900
-Wire Wire Line
-	8600 3750 8100 3750
-Wire Wire Line
 	8550 3550 8600 3550
 Wire Wire Line
@@
 	1    0    0    -1
 $EndComp
+Wire Wire Line
+	8600 3850 7650 3850
+Wire Wire Line
+	7050 2900 7750 2900
+Wire Wire Line
+	7750 2900 7750 3750
+Wire Wire Line
+	7750 3750 8600 3750
+Wire Wire Line
+	7650 3850 7650 3900
+Wire Wire Line
+	7650 3900 7050 3900
+Wire Wire Line
+	5250 3300 5550 3300
+Wire Wire Line
+	5850 3900 5550 3900
+Wire Wire Line
+	5550 3300 5550 3900
+Connection ~ 5550 3900
+Wire Wire Line
+	5550 3900 5550 4000
+Wire Wire Line
+	5250 3500 5350 3500
+Wire Wire Line
+	5350 3500 5350 2900
+Wire Wire Line
+	5350 2900 5550 2900
+Connection ~ 5550 2900
+Wire Wire Line
+	5550 2900 5850 2900
 $EndSCHEMATC
